Commit message: Parameterize ros2_control hardware plugin in launch and xacro files
Enable customization of `ros2_control` URDF
`<hardware><plugin/></hardware>` tag contents through launch file
parameters.

Other projects extending the demos may introduce their own hardware
interfaces in this way.

File: example_1/description/ros2_control/rrbot.ros2_control.xacro (robot description, xacro)
@@ -1,8 +1,8 @@
 <?xml version="1.0"?>
 <robot xmlns:xacro="http://www.ros.org/wiki/xacro">
-  <xacro:macro name="rrbot_ros2_control" params="name prefix">
+  <xacro:macro name="rrbot_ros2_control" params="name prefix hardware_plugin">
     <ros2_control name="${name}" type="system">
       <hardware>
-        <plugin>ros2_control_demo_example_1/RRBotSystemPositionOnlyHardware</plugin>
+        <plugin>${hardware_plugin}</plugin>
         <param name="example_param_hw_start_duration_sec">0</param>
         <param name="example_param_hw_stop_duration_sec">3.0</param>

File: example_1/description/urdf/rrbot.urdf.xacro (robot description, xacro)
@@ -7,4 +7,6 @@
 <robot xmlns:xacro="http://www.ros.org/wiki/xacro" name="2dof_robot">
   <xacro:arg name="prefix" default="" />
+  <xacro:arg name="hardware_plugin"
+             default="ros2_control_demo_example_1/RRBotSystemPositionOnlyHardware" />
   <!-- Import RRBot macro -->
   <xacro:include filename="$(find ros2_control_demo_example_1)/urdf/rrbot_description.urdf.xacro" />
@@ -19,4 +21,5 @@
   </xacro:rrbot>
   <xacro:rrbot_ros2_control
-    name="RRBot" prefix="$(arg prefix)" />
+    name="RRBot" prefix="$(arg prefix)"
+    hardware_plugin="$(arg hardware_plugin)" />
 </robot>

File: example_2/description/ros2_control/diffbot.ros2_control.xacro (robot description, xacro)
@@ -4,5 +4,5 @@
     <ros2_control name="${name}" type="system">
       <hardware>
-        <plugin>ros2_control_demo_example_2/DiffBotSystemHardware</plugin>
+        <plugin>${hardware_plugin}</plugin>
         <param name="example_param_hw_start_duration_sec">0</param>
         <param name="example_param_hw_stop_duration_sec">3.0</param>

File: example_2/description/urdf/diffbot.urdf.xacro (robot description, xacro)
@@ -3,4 +3,6 @@
 <robot xmlns:xacro="http://www.ros.org/wiki/xacro" name="diffdrive_robot">
   <xacro:arg name="prefix" default="" />
+  <xacro:arg name="hardware_plugin"
+             default="ros2_control_demo_example_2/DiffBotSystemHardware" />
   <xacro:include filename="$(find ros2_control_demo_example_2)/urdf/diffbot_description.urdf.xacro" />
   <!-- Import Rviz colors -->
@@ -10,4 +12,5 @@
   <xacro:diffbot prefix="$(arg prefix)" />
   <xacro:diffbot_ros2_control
-    name="DiffBot" prefix="$(arg prefix)" />
+    name="DiffBot" prefix="$(arg prefix)"
+    hardware_plugin="$(arg hardware_plugin)" />
 </robot>

File: example_3/description/ros2_control/rrbot_system_multi_interface.ros2_control.xacro (robot description, xacro)
@@ -1,5 +1,5 @@
 <?xml version="1.0"?>
 <robot xmlns:xacro="http://www.ros.org/wiki/xacro">
-  <xacro:macro name="rrbot_system_multi_interface" params="name prefix use_mock_hardware:=^|true mock_sensor_commands:=^|false slowdown:=2.0">
+  <xacro:macro name="rrbot_system_multi_interface" params="name prefix use_mock_hardware:=^|true mock_sensor_commands:=^|false slowdown:=2.0 hardware_plugin:=^|null">
     <ros2_control name="${name}" type="system">
       <hardware>
@@ -10,5 +10,5 @@
         </xacro:if>
         <xacro:unless value="${use_mock_hardware}">
-          <plugin>ros2_control_demo_example_3/RRBotSystemMultiInterfaceHardware</plugin>
+          <plugin>${hardware_plugin}</plugin>
           <param name="example_param_hw_start_duration_sec">0.0</param>
           <param name="example_param_hw_stop_duration_sec">3.0</param>

File: example_3/description/urdf/rrbot_system_multi_interface.urdf.xacro (robot description, xacro)
@@ -9,4 +9,6 @@
   <xacro:arg name="use_mock_hardware" default="false" />
   <xacro:arg name="mock_sensor_commands" default="false" />
+  <xacro:arg name="hardware_plugin"
+             default="ros2_control_demo_example_3/RRBotSystemMultiInterfaceHardware" />
   <xacro:arg name="prefix" default="" />
   <xacro:arg name="slowdown" default="100.0" />
@@ -26,4 +28,5 @@
     use_mock_hardware="$(arg use_mock_hardware)"
     mock_sensor_commands="$(arg mock_sensor_commands)"
+    hardware_plugin="$(arg hardware_plugin)"
     slowdown="$(arg slowdown)" />
 </robot>

File: example_4/description/ros2_control/rrbot_system_with_sensor.ros2_control.xacro (robot description, xacro)
@@ -1,5 +1,5 @@
 <?xml version="1.0"?>
 <robot xmlns:xacro="http://www.ros.org/wiki/xacro">
-  <xacro:macro name="rrbot_system_with_sensor" params="name prefix use_mock_hardware:=^|true mock_sensor_commands:=^|false slowdown:=2.0">
+  <xacro:macro name="rrbot_system_with_sensor" params="name prefix use_mock_hardware:=^|true mock_sensor_commands:=^|false slowdown:=2.0 hardware_plugin:=^|null">
     <ros2_control name="${name}" type="system">
       <hardware>
@@ -10,5 +10,5 @@
         </xacro:if>
         <xacro:unless value="${use_mock_hardware}">
-          <plugin>ros2_control_demo_example_4/RRBotSystemWithSensorHardware</plugin>
+          <plugin>${hardware_plugin}</plugin>
           <param name="example_param_hw_start_duration_sec">0.0</param>
           <param name="example_param_hw_stop_duration_sec">3.0</param>

File: example_4/description/urdf/rrbot_system_with_sensor.urdf.xacro (robot description, xacro)
@@ -9,4 +9,6 @@
   <xacro:arg name="use_mock_hardware" default="false" />
   <xacro:arg name="mock_sensor_commands" default="false" />
+  <xacro:arg name="hardware_plugin"
+             default="ros2_control_demo_example_4/RRBotSystemWithSensorHardware" />
   <xacro:arg name="prefix" default="" />
   <xacro:arg name="slowdown" default="50.0" />
@@ -26,4 +28,5 @@
     use_mock_hardware="$(arg use_mock_hardware)"
     mock_sensor_commands="$(arg mock_sensor_commands)"
+    hardware_plugin="$(arg hardware_plugin)"
     slowdown="$(arg slowdown)" />
 </robot>

File: example_5/description/ros2_control/external_rrbot_force_torque_sensor.ros2_control.xacro (robot description, xacro)
@@ -1,5 +1,5 @@
 <?xml version="1.0"?>
 <robot xmlns:xacro="http://www.ros.org/wiki/xacro">
-  <xacro:macro name="external_rrbot_force_torque_sensor" params="name prefix use_mock_hardware:=^|true mock_sensor_commands:=^|false">
+  <xacro:macro name="external_rrbot_force_torque_sensor" params="name prefix use_mock_hardware:=^|true mock_sensor_commands:=^|false hardware_plugin:=^|null">
     <ros2_control name="${name}" type="sensor">
       <hardware>
@@ -10,5 +10,5 @@
         </xacro:if>
         <xacro:unless value="${use_mock_hardware}">
-          <plugin>ros2_control_demo_example_5/ExternalRRBotForceTorqueSensorHardware</plugin>
+          <plugin>${hardware_plugin}</plugin>
           <param name="example_param_hw_start_duration_sec">0.0</param>
           <param name="example_param_hw_stop_duration_sec">3.0</param>

File: example_5/description/ros2_control/rrbot_system_position_only.ros2_control.xacro (robot description, xacro)
@@ -1,5 +1,5 @@
 <?xml version="1.0"?>
 <robot xmlns:xacro="http://www.ros.org/wiki/xacro">
-  <xacro:macro name="rrbot_system_position_only" params="name prefix use_mock_hardware:=^|true mock_sensor_commands:=^|false slowdown:=2.0">
+  <xacro:macro name="rrbot_system_position_only" params="name prefix use_mock_hardware:=^|true mock_sensor_commands:=^|false slowdown:=2.0 hardware_plugin:=^|null">
     <ros2_control name="${name}" type="system">
       <hardware>
@@ -10,5 +10,5 @@
         </xacro:if>
         <xacro:unless value="${use_mock_hardware}">
-          <plugin>ros2_control_demo_example_5/RRBotSystemPositionOnlyHardware</plugin>
+          <plugin>${hardware_plugin}</plugin>
           <param name="example_param_hw_start_duration_sec">0.0</param>
           <param name="example_param_hw_stop_duration_sec">3.0</param>

File: example_5/description/urdf/rrbot_system_with_external_sensor.urdf.xacro (robot description, xacro)
@@ -9,4 +9,8 @@
   <xacro:arg name="use_mock_hardware" default="true" />
   <xacro:arg name="mock_sensor_commands" default="false" />
+  <xacro:arg name="hardware_position_plugin"
+             default="ros2_control_demo_example_5/RRBotSystemPositionOnlyHardware" />
+  <xacro:arg name="hardware_sensor_plugin"
+             default="ros2_control_demo_example_5/ExternalRRBotForceTorqueSensorHardware" />
   <xacro:arg name="prefix" default="" />
   <xacro:arg name="slowdown" default="50.0" />
@@ -28,8 +32,10 @@
     use_mock_hardware="$(arg use_mock_hardware)"
     mock_sensor_commands="$(arg mock_sensor_commands)"
+    hardware_plugin="$(arg hardware_position_plugin)"
     slowdown="$(arg slowdown)" />
   <xacro:external_rrbot_force_torque_sensor
     name="ExternalRRBotFTSensor" prefix="$(arg prefix)"
     use_mock_hardware="$(arg use_mock_hardware)"
-    mock_sensor_commands="$(arg mock_sensor_commands)" />
+    mock_sensor_commands="$(arg mock_sensor_commands)"
+    hardware_plugin="$(arg hardware_sensor_plugin)" />
 </robot>

File: example_6/description/ros2_control/rrbot_modular_actuators.ros2_control.xacro (robot description, xacro)
@@ -1,8 +1,8 @@
 <?xml version="1.0"?>
 <robot xmlns:xacro="http://www.ros.org/wiki/xacro">
-  <xacro:macro name="rrbot_modular_actuators" params="name prefix slowdown:=2.0">
+  <xacro:macro name="rrbot_modular_actuators" params="name prefix slowdown:=2.0 hardware_plugin">
     <ros2_control name="RRBotModularJoint1" type="actuator">
       <hardware>
-        <plugin>ros2_control_demo_example_6/RRBotModularJoint</plugin>
+        <plugin>${hardware_plugin}</plugin>
         <param name="example_param_hw_start_duration_sec">2.0</param>
         <param name="example_param_hw_stop_duration_sec">3.0</param>
@@ -19,5 +19,5 @@
     <ros2_control name="RRBotModularJoint2" type="actuator">
       <hardware>
-        <plugin>ros2_control_demo_example_6/RRBotModularJoint</plugin>
+        <plugin>${hardware_plugin}</plugin>
         <param name="example_param_hw_start_duration_sec">2.0</param>
         <param name="example_param_hw_stop_duration_sec">3.0</param>

File: example_6/description/urdf/rrbot_modular_actuators.urdf.xacro (robot description, xacro)
@@ -9,4 +9,6 @@
   <xacro:arg name="prefix" default="" />
   <xacro:arg name="slowdown" default="2.0" />
+  <xacro:arg name="hardware_plugin"
+             default="ros2_control_demo_example_6/RRBotModularJoint" />
   <!-- Import RRBot macro -->
   <xacro:include filename="$(find ros2_control_demo_example_6)/urdf/rrbot_description.urdf.xacro" />
@@ -22,4 +24,5 @@
   <xacro:rrbot_modular_actuators
     name="RRBotModularJoint" prefix="$(arg prefix)"
+    hardware_plugin="$(arg hardware_plugin)"
     slowdown="$(arg slowdown)" />
 </robot>

File: example_8/description/ros2_control/rrbot_transmissions_system_position_only.ros2_control.xacro (robot description, xacro)
@@ -1,8 +1,8 @@
 <?xml version="1.0"?>
 <robot xmlns:xacro="http://www.ros.org/wiki/xacro">
-  <xacro:macro name="rrbot_transmissions_system_position_only" params="name prefix slowdown:=2.0">
+  <xacro:macro name="rrbot_transmissions_system_position_only" params="name prefix slowdown:=2.0 hardware_plugin">
     <ros2_control name="${name}" type="system">
       <hardware>
-        <plugin>ros2_control_demo_example_8/RRBotTransmissionsSystemPositionOnlyHardware</plugin>
+        <plugin>${hardware_plugin}</plugin>
         <param name="actuator_slowdown">${slowdown}</param>
       </hardware>

File: example_8/description/urdf/rrbot_transmissions_system_position_only.urdf.xacro (robot description, xacro)
@@ -8,4 +8,6 @@
   <!-- Enable setting arguments from the launch file -->
   <xacro:arg name="prefix" default="" />
+  <xacro:arg name="hardware_plugin"
+             default="ros2_control_demo_example_8/RRBotTransmissionsSystemPositionOnlyHardware" />
   <xacro:arg name="slowdown" default="100.0" />
   <!-- Import RRBot macro -->
@@ -22,4 +24,5 @@
   <xacro:rrbot_transmissions_system_position_only
     name="RRBotTransmissionsSystemPositionOnly" prefix="$(arg prefix)"
+    hardware_plugin="$(arg hardware_plugin)"
     slowdown="$(arg slowdown)" />
 </robot>
