Commit message: Parameterize ros2_control hardware plugin in launch and xacro files
Enable customization of `ros2_control` URDF
`<hardware><plugin/></hardware>` tag contents through launch file
parameters.

Other projects extending the demos may introduce their own hardware
interfaces in this way.

File: ros2_control_demo_description/rrbot_description/ros2_control/rrbot.ros2_control.xacro (robot description, xacro)
@@ -1,8 +1,8 @@
 <?xml version="1.0"?>
 <robot xmlns:xacro="http://www.ros.org/wiki/xacro">
-  <xacro:macro name="rrbot_ros2_control" params="name prefix">
+  <xacro:macro name="rrbot_ros2_control" params="name prefix hardware_plugin:=^|ros2_control_demo_hardware/RRBotSystemPositionOnlyHardware">
     <ros2_control name="${name}" type="system">
       <hardware>
-        <plugin>ros2_control_demo_hardware/RRBotSystemPositionOnlyHardware</plugin>
+        <plugin>${hardware_plugin}</plugin>
         <param name="example_param_hw_start_duration_sec">0</param>
         <param name="example_param_hw_stop_duration_sec">3.0</param>

File: ros2_control_demo_description/rrbot_description/ros2_control/rrbot_system_multi_interface.ros2_control.xacro (robot description, xacro)
@@ -1,5 +1,5 @@
 <?xml version="1.0"?>
 <robot xmlns:xacro="http://www.ros.org/wiki/xacro">
-  <xacro:macro name="rrbot_system_multi_interface" params="name prefix use_sim:=^|false use_fake_hardware:=^|true fake_sensor_commands:=^|false slowdown:=2.0">
+  <xacro:macro name="rrbot_system_multi_interface" params="name prefix use_sim:=^|false use_fake_hardware:=^|true fake_sensor_commands:=^|false slowdown:=2.0 hardware_plugin:=^|ros2_control_demo_hardware/RRBotSystemMultiInterfaceHardware">
     <ros2_control name="${name}" type="system">
       <xacro:if value="$(arg use_sim)">
@@ -16,5 +16,5 @@
           </xacro:if>
           <xacro:unless value="${use_fake_hardware}">
-            <plugin>ros2_control_demo_hardware/RRBotSystemMultiInterfaceHardware</plugin>
+            <plugin>${hardware_plugin}</plugin>
             <param name="example_param_hw_start_duration_sec">2.0</param>
             <param name="example_param_hw_stop_duration_sec">3.0</param>

File: ros2_control_demo_description/rrbot_description/ros2_control/rrbot_system_position_only.ros2_control.xacro (robot description, xacro)
@@ -1,5 +1,5 @@
 <?xml version="1.0"?>
 <robot xmlns:xacro="http://www.ros.org/wiki/xacro">
-  <xacro:macro name="rrbot_system_position_only" params="name prefix use_sim:=^|false use_fake_hardware:=^|true fake_sensor_commands:=^|false slowdown:=2.0">
+  <xacro:macro name="rrbot_system_position_only" params="name prefix use_sim:=^|false use_fake_hardware:=^|true fake_sensor_commands:=^|false slowdown:=2.0 hardware_plugin:=^|ros2_control_demo_hardware/RRBotSystemPositionOnlyHardware">
     <ros2_control name="${name}" type="system">
       <xacro:if value="$(arg use_sim)">
@@ -16,5 +16,5 @@
           </xacro:if>
           <xacro:unless value="${use_fake_hardware}">
-            <plugin>ros2_control_demo_hardware/RRBotSystemPositionOnlyHardware</plugin>
+            <plugin>${hardware_plugin}</plugin>
             <param name="example_param_hw_start_duration_sec">2.0</param>
             <param name="example_param_hw_stop_duration_sec">3.0</param>

File: ros2_control_demo_description/rrbot_description/ros2_control/rrbot_system_with_sensor.ros2_control.xacro (robot description, xacro)
@@ -1,5 +1,5 @@
 <?xml version="1.0"?>
 <robot xmlns:xacro="http://www.ros.org/wiki/xacro">
-  <xacro:macro name="rrbot_system_with_sensor" params="name prefix use_sim:=^|false use_fake_hardware:=^|true fake_sensor_commands:=^|false slowdown:=2.0">
+  <xacro:macro name="rrbot_system_with_sensor" params="name prefix use_sim:=^|false use_fake_hardware:=^|true fake_sensor_commands:=^|false slowdown:=2.0 hardware_plugin:=^|ros2_control_demo_hardware/RRBotSystemWithSensorHardware">
     <ros2_control name="${name}" type="system">
       <hardware>
@@ -10,5 +10,5 @@
         </xacro:if>
         <xacro:unless value="${use_fake_hardware}">
-          <plugin>ros2_control_demo_hardware/RRBotSystemWithSensorHardware</plugin>
+          <plugin>${hardware_plugin}</plugin>
           <param name="example_param_hw_start_duration_sec">0.0</param>
           <param name="example_param_hw_stop_duration_sec">3.0</param>

File: ros2_control_demo_description/rrbot_description/urdf/rrbot.urdf.xacro (robot description, xacro)
@@ -7,4 +7,6 @@
 <robot xmlns:xacro="http://www.ros.org/wiki/xacro" name="2dof_robot">
   <xacro:arg name="prefix" default="" />
+  <xacro:arg name="hardware_plugin"
+             default="ros2_control_demo_hardware/RRBotSystemPositionOnlyHardware" />
   <!-- Import RRBot macro -->
   <xacro:include filename="$(find rrbot_description)/urdf/rrbot_description.urdf.xacro" />
@@ -22,4 +24,5 @@
   </xacro:rrbot>
   <xacro:rrbot_ros2_control
-    name="RRBot" prefix="$(arg prefix)" />
+    name="RRBot" prefix="$(arg prefix)"
+    hardware_plugin="$(arg hardware_plugin)" />
 </robot>

File: ros2_control_demo_description/rrbot_description/urdf/rrbot_system_multi_interface.urdf.xacro (robot description, xacro)
@@ -8,4 +8,6 @@
   <xacro:arg name="use_sim" default="false" />
   <!-- Enable setting arguments from the launch file -->
+  <xacro:arg name="hardware_plugin"
+             default="ros2_control_demo_hardware/RRBotSystemMultiInterfaceHardware" />
   <xacro:arg name="use_fake_hardware" default="false" />
   <xacro:arg name="fake_sensor_commands" default="false" />
@@ -31,4 +33,5 @@
   <xacro:rrbot_system_multi_interface
     name="RRBotSystemMultiInterface" prefix="$(arg prefix)"
+    hardware_plugin="$(arg hardware_plugin)"
     use_fake_hardware="$(arg use_fake_hardware)"
     fake_sensor_commands="$(arg fake_sensor_commands)"

File: ros2_control_demo_description/rrbot_description/urdf/rrbot_system_position_only.urdf.xacro (robot description, xacro)
@@ -8,4 +8,6 @@
   <xacro:arg name="use_sim" default="false" />
   <!-- Enable setting arguments from the launch file -->
+  <xacro:arg name="hardware_plugin"
+             default="ros2_control_demo_hardware/RRBotSystemPositionOnlyHardware" />
   <xacro:arg name="use_fake_hardware" default="false" />
   <xacro:arg name="fake_sensor_commands" default="false" />
@@ -31,4 +33,5 @@
   <xacro:rrbot_system_position_only
     name="RRBotSystemPositionOnly" prefix="$(arg prefix)"
+    hardware_plugin="$(arg hardware_plugin)"
     use_fake_hardware="$(arg use_fake_hardware)"
     fake_sensor_commands="$(arg fake_sensor_commands)"

File: ros2_control_demo_description/rrbot_description/urdf/rrbot_system_with_sensor.urdf.xacro (robot description, xacro)
@@ -8,4 +8,6 @@
   <xacro:arg name="use_sim" default="false" />
   <!-- Enable setting arguments from the launch file -->
+  <xacro:arg name="hardware_plugin"
+             default="ros2_control_demo_hardware/RRBotSystemWithSensorHardware" />
   <xacro:arg name="use_fake_hardware" default="false" />
   <xacro:arg name="fake_sensor_commands" default="false" />
@@ -28,4 +30,5 @@
   <xacro:rrbot_system_with_sensor
     name="RRBotSystemWithSensor" prefix="$(arg prefix)"
+    hardware_plugin="$(arg hardware_plugin)"
     use_fake_hardware="$(arg use_fake_hardware)"
     fake_sensor_commands="$(arg fake_sensor_commands)"
